Commit message: tmp

File: pma_description/config/pma_planar_2dof.ros2_control.xacro (robot description, xacro)
@@ -2,5 +2,4 @@
 <robot xmlns:xacro="http://www.ros.org/wiki/xacro">
     <xacro:macro name="pma_planar_2dof_ros2_control" params="name initial_positions_file">
-        <xacro:property name="initial_positions" value="${load_yaml(initial_positions_file)['initial_positions']}"/>
         <ros2_control name="${name}" type="system">
             <hardware>
@@ -9,14 +8,8 @@
             <joint name="pma_planar_2dof_shoulder">
                 <command_interface name="pressure"/>
-                <state_interface name="position">
-                  <param name="initial_value">${initial_positions['pma_planar_2dof_shoulder']}</param>
-                </state_interface>
                 <state_interface name="pressure"/>
             </joint>
             <joint name="pma_planar_2dof_elbow">
                 <command_interface name="pressure"/>
-                <state_interface name="position">
-                  <param name="initial_value">${initial_positions['pma_planar_2dof_elbow']}</param>
-                </state_interface>
                 <state_interface name="pressure"/>
             </joint>
